File: PCB Files/Power Core Board/Lightsaber Power Core/Lightsaber Power Core.kicad_sch (KiCad schematic)
At the start: 4 parts

Commit message: Checkpoint before removing VEXT switches
Parts:
- removed U?: STM32L431RCTx, Package_QFP:LQFP-64_10x10mm_P0.5mm, symbol MCU_ST_STM32L4:STM32L431RCTx
- added C? (x6): 0.1uF, symbol Device:C
- added C? (x8): 1uF, symbol Device:C
- added C? (x2): 22uF, symbol Device:C
- added J1: BM02B-ACHSS-GAN-ETF, Connector_JST:JST_ACH_BM02B-ACHSS-GAN-ETF_1x02-1MP_P1.20mm_Vertical, symbol Connector_Generic_MountingPin:Conn_01x02_MountingPin
- added J?: SWD, symbol Connector_Generic:Conn_02x05_Odd_Even
- added J?: Interface Connector, symbol Connector:Screw_Terminal_01x05
- added J?: UART, symbol Connector_Generic:Conn_01x03
- added JP? (x2): Cut Jump, symbol Jumper:SolderJumper_2_Bridged
- added LABELPORT? (x23): SHORT_NET_NAME(1), symbol irex_Drawing_Symbols:Port_Input_NoNetName
- added LABELPORT? (x16): SHORT_NET_NAME(1), symbol irex_Drawing_Symbols:Port_I/O_NoNetName
- added LABELPORT? (x23): SHORT_NET_NAME(1), symbol irex_Drawing_Symbols:Port_Output_NoNetName
- added Q?: AO3401A, symbol Device:Q_PMOS_GSD
- added Q?: 2302V, symbol Device:Q_NMOS_GSD
- added R? (x3): 634k, symbol Device:R_US
- added R? (x8): 10k, symbol Device:R_US
- added R? (x3): 200, symbol Device:R_US
- added R? (x3): 2k, symbol Device:R_US
- added R? (x4): 0, symbol Device:R_US
- added R?: 100, symbol Device:R_US
- added SW?: MCU Reset, symbol Switch:SW_Push
- added SW?: MCU Boot, symbol Switch:SW_Push
- added U?: STM32L452CCUx, Package_DFN_QFN:QFN-48-1EP_7x7mm_P0.5mm_EP5.6x5.6mm, symbol MCU_ST_STM32L4:STM32L452CCUx
Connections:
- net at U?.A1 (~{SD_MODE}): now also R?.1
- net 5.0V: now reaches U?.A2 (VDD)
- net 5.0V: now also C?.1, C?.1, Q?.2 (S), R?.2
- net SPK+: now reaches U?.A3 (OUTP)
- net SPK+: now also J?.5 (Pin_5), LABELPORT?.1 (IN), LABELPORT?.1 (OUT)
- net at U?.B1 (DIN): now also R?.1
- net GND: now reaches U?.B2 (GAIN_SLOT)
- net GND: now also U?.2 (SDx), U?.3 (SCx), U?.4 (GND), U?.6 (GND), U?.7 (GND), U?.C2 (GND), C?.2, C?.2, C?.2, C?.2, C?.2, C?.2, C?.2, C?.2, C?.2, C?.2, C?.2, C?.2, C?.2, C?.2, C?.2, C?.2, J1.2 (Pin_2), J1.MP (MountPin), J?.1 (Pin_1), J?.1 (Pin_1), J?.3 (Pin_3), J?.5 (Pin_5), J?.9 (Pin_9), Q?.2 (S), R?.1, R?.1, R?.1, R?.1, SW?.1, U?.23 (VSS), U?.35 (VSS), U?.47 (VSS), U?.49 (VSS), U?.8 (VSSA)
- net SPK-: now reaches U?.B3 (OUTN)
- net SPK-: now also J?.4 (Pin_4), LABELPORT?.1 (IN), LABELPORT?.1 (OUT)
- net at U?.C1 (BCLK): now also R?.1
- net at U?.C3 (LRCLK): now also R?.1
- net at U?.1 (SDO/SA0): now also R?.1, R?.1, R?.2
- net at U?.12 (~{CS}): now also R?.1, R?.2
- net I2C2_SCL/SPI2_SCK: now reaches U?.13 (SCL)
- net I2C2_SCL/SPI2_SCK: now also LABELPORT?.1 (IN), LABELPORT?.1 (OUT), R?.1, U?.21 (PB10)
- net at U?.14 (SDA): now also R?.1, R?.1, R?.1
- net IMU_INT1: now reaches U?.4 (INT1)
- net IMU_INT1: now also LABELPORT?.1 (OUT)
- net 3.3V: now reaches U?.5 (VDDIO)
- net 3.3V: now also U?.8 (VCC), U?.8 (VDD), C?.1, C?.1, C?.1, C?.1, C?.1, C?.1, C?.1, C?.1, J?.1 (Pin_1), JP?.2 (B), JP?.2 (B), R?.1, R?.2, R?.2, R?.2, R?.2, U?.1 (VBAT), U?.24 (VDD), U?.48 (VDD)
- net QSPI_~{CS}: now reaches U?.1 (~{CS})
- net QSPI_~{CS}: now also LABELPORT?.1 (IN), LABELPORT?.1 (OUT), U?.12 (PA2)
- net QSPI_IO1: now reaches U?.2 (DO(IO1))
- net QSPI_IO1: now also LABELPORT?.1 (I/O), LABELPORT?.1 (I/O), U?.18 (PB0)
- net QSPI_IO2: now reaches U?.3 (~{WP}/IO2)
- net QSPI_IO2: now also LABELPORT?.1 (I/O), LABELPORT?.1 (I/O), U?.17 (PA7)
- net QSPI_IO0: now reaches U?.5 (DI(IO0))
- net QSPI_IO0: now also LABELPORT?.1 (I/O), LABELPORT?.1 (I/O), U?.19 (PB1)
- net QSPI_CLK: now reaches U?.6 (CLK)
- net QSPI_CLK: now also LABELPORT?.1 (IN), LABELPORT?.1 (OUT), U?.13 (PA3)
- net QSPI_IO3: now reaches U?.7 (~{HOLD}/IO3)
- net QSPI_IO3: now also LABELPORT?.1 (I/O), LABELPORT?.1 (I/O), U?.16 (PA6)
- new net: R?.1, SW?.2 (x2)
- new net: Q?.1 (G), Q?.3 (D), R?.1
- new net: J1.1 (Pin_1), R?.1
- new net 3.3V_EN: LABELPORT?.1 (IN)
- new net 5.0V_EN: LABELPORT?.1 (IN), LABELPORT?.1 (OUT), U?.4 (PC15)
- new net 5.0V_SW: C?.1, J?.3 (Pin_3), Q?.3 (D)
- new net 5.0V_SW_EN: LABELPORT?.1 (IN), LABELPORT?.1 (OUT), Q?.1 (G), R?.2, U?.6 (PH1)
- new net AUDIO_BLCK: LABELPORT?.1 (IN), LABELPORT?.1 (OUT), R?.2, U?.29 (PA8)
- new net AUDIO_DIN: LABELPORT?.1 (IN), LABELPORT?.1 (OUT), R?.2, U?.31 (PA10)
- new net AUDIO_LRCLK: LABELPORT?.1 (IN), LABELPORT?.1 (OUT), R?.2, U?.30 (PA9)
- new net AUDIO_~{SD_MODE}: LABELPORT?.1 (IN), LABELPORT?.1 (OUT), R?.2, U?.5 (PH0)
- new net BOOT0: R?.2, SW?.1, U?.44 (PH3)
- new net BTN_WKUP: C?.1, LABELPORT?.1 (IN), LABELPORT?.1 (OUT), R?.2, U?.10 (PA0)
- new net CHARGE_STAT: LABELPORT?.1 (IN), LABELPORT?.1 (OUT), U?.2 (PC13)
- new net I2C2_SDA: LABELPORT?.1 (I/O), LABELPORT?.1 (I/O), R?.2, U?.22 (PB11)
- new net MCU_~{RST}: C?.1, J?.10 (Pin_10), LABELPORT?.1 (IN), LABELPORT?.1 (OUT), R?.2, U?.7 (NRST)
- new net SPI2_MISO: LABELPORT?.1 (IN), LABELPORT?.1 (OUT), R?.2, U?.27 (PB14)
- new net SPI2_MOSI: LABELPORT?.1 (IN), LABELPORT?.1 (OUT), R?.2, U?.28 (PB15)
- new net SPI2_NSS: LABELPORT?.1 (IN), LABELPORT?.1 (OUT), R?.2, U?.25 (PB12)
- new net SWCLK: J?.4 (Pin_4), LABELPORT?.1 (IN), LABELPORT?.1 (OUT), U?.37 (PA14)
- new net SWDIO: J?.2 (Pin_2), LABELPORT?.1 (I/O), LABELPORT?.1 (I/O), U?.34 (PA13)
- new net SWO: J?.6 (Pin_6), LABELPORT?.1 (IN), LABELPORT?.1 (OUT), U?.39 (PB3)
- new net UART_MCU_RX: J?.2 (Pin_2), LABELPORT?.1 (IN), LABELPORT?.1 (OUT), U?.43 (PB7)
- new net UART_MCU_TX: J?.3 (Pin_3), LABELPORT?.1 (IN), LABELPORT?.1 (OUT), U?.42 (PB6)
- new net USB_DM: LABELPORT?.1 (I/O), U?.32 (PA11)
- new net USB_DN: LABELPORT?.1 (I/O)
- new net USB_DP: LABELPORT?.1 (I/O), LABELPORT?.1 (I/O), U?.33 (PA12)
- new net VDDA: C?.1, C?.1, JP?.1 (A), U?.9 (VDDA)
- new net VDDUSB: C?.1, JP?.1 (A), U?.36 (VDDUSB)
- new net VSYS: R?.2
- new net VSYS_SENSE: R?.1, R?.2, U?.11 (PA1)
- new net WS2812_DATA: LABELPORT?.1 (IN), LABELPORT?.1 (OUT), R?.2, U?.15 (PA5)
- new net WS2812_DOUT: J?.2 (Pin_2), R?.1
- no-connect marks 0 -> 5
Other:
- note added: "Audio Driver"
- note added: "Flash"
- note added: "IMU"
- note added: "Power Button Connector"
- note added: "Program/Debug"
- note added: "Terminal Block"
- moved on the sheet: U?

Commit message: Schematic drawn, ready for post-wiring
Parts:
- removed C? (x5): 0.1uF, symbol Device:C
- removed C? (x8): 1uF, symbol Device:C
- removed C?: 22uF, symbol Device:C
- removed J?: SWD, symbol Connector_Generic:Conn_02x05_Odd_Even
- removed J?: UART, symbol Connector_Generic:Conn_01x03
- removed JP? (x2): Cut Jump, symbol Jumper:SolderJumper_2_Bridged
- removed LABELPORT? (x23): SHORT_NET_NAME(1), symbol irex_Drawing_Symbols:Port_Input_NoNetName
- removed LABELPORT? (x16): SHORT_NET_NAME(1), symbol irex_Drawing_Symbols:Port_I/O_NoNetName
- removed LABELPORT? (x23): SHORT_NET_NAME(1), symbol irex_Drawing_Symbols:Port_Output_NoNetName
- removed R? (x3): 634k, symbol Device:R_US
- removed R? (x5): 10k, symbol Device:R_US
- removed R? (x3): 200, symbol Device:R_US
- removed R? (x3): 2k, symbol Device:R_US
- removed R? (x4): 0, symbol Device:R_US
- removed SW?: MCU Reset, symbol Switch:SW_Push
- removed SW?: MCU Boot, symbol Switch:SW_Push
- removed U?: MAX98357xW, Package_BGA:WLP-9_1.448x1.468mm_Layout3x3_P0.4mm_Ball0.27mm_Pad0.25mm, symbol irex_Amplifier_Audio:MAX98357xW
- removed U?: LSM6DSR, Package_LGA:LGA-14_3x2.5mm_P0.5mm_LayoutBorder3x4y, symbol irex_Sensor_Motion:LSM6DSR
- removed U?: STM32L452CCUx, Package_DFN_QFN:QFN-48-1EP_7x7mm_P0.5mm_EP5.6x5.6mm, symbol MCU_ST_STM32L4:STM32L452CCUx
- removed U?: W25N01GVZE, Package_SON:WSON-8-1EP_8x6mm_P1.27mm_EP3.4x4.3mm, symbol irex_Memory_Flash:W25N01GVZE
- added C?: 22uF, symbol Device:C
- added C? (x2): 10uF, symbol Device:C
- added J?: SWD, symbol Connector_Generic:Conn_02x05_Odd_Even
- added J?: USB-C, symbol Connector:USB_C_Receptacle_USB2.0_16P
- added J?: VBAT, symbol Connector:Screw_Terminal_01x02
- added J?: UART, symbol Connector_Generic:Conn_01x03
- added NT?: VBAT_LED, symbol Device:NetTie_2
- added Q?: XR25P01M, symbol Device:Q_PMOS_GSD
- added R? (x2): 5.1k, symbol Device:R_US
- added TP?: 3V3EN, symbol Connector:TestPoint
- added U?: CM1213A−02Sx, symbol irex_Power_Protection:CM1213A−02Sx
- Q?: value AO3401A -> XR25P01M; LCSC PN (none) -> C42456887; MPN (none) -> XR25P01M
Connections:
- net 3.3V: now also J?.1 (Pin_1)
- net 3.3V_EN: now also TP?.1
- net GND: now also C?.2, C?.2, C?.2, J?.1 (Pin_1), J?.2 (Pin_2), J?.3 (Pin_3), J?.5 (Pin_5), J?.9 (Pin_9), J?.A1 (GND), J?.A12 (GND), J?.B1 (GND), J?.B12 (GND), J?.S1 (SHIELD), R?.2, R?.2, U?.1 (VN)
- net MCU_~{RST}: now also J?.10 (Pin_10)
- net SWCLK: now also J?.4 (Pin_4)
- net SWDIO: now also J?.2 (Pin_2)
- net SWO: now also J?.6 (Pin_6)
- net UART_MCU_RX: now also J?.2 (Pin_2)
- net UART_MCU_TX: now also J?.3 (Pin_3)
- net USB_DN: now also J?.A7 (D-), J?.B7 (D-), U?.2 (CH1)
- net USB_DP: now also J?.A6 (D+), J?.B6 (D+), U?.3 (CH2)
- net at Q?.1 (G), Q?.3 (D), R?.1: now also Q?.1 (G)
- net 5.0V renamed VBAT_LED
- net VBAT_LED: now also C?.1, J?.1 (Pin_1), NT?.1, Q?.2 (S)
- net 5.0V_SW renamed VBAT_LED_SW
- net VBAT_LED_SW: now also C?.1, Q?.3 (D)
- net 5.0V_SW_EN renamed VBAT_LED_SW_EN
- new net: J?.B5 (CC2), R?.1
- new net: J?.A5 (CC1), R?.1
- new net VBAT: NT?.2
- new net VBUS: C?.1, J?.A4 (VBUS), J?.A9 (VBUS), J?.B4 (VBUS), J?.B9 (VBUS), U?.4 (VP)
- no-connect marks 5 -> 4
Other:
- added sheet MCU & Peripheral (mcu_and_peripheral.kicad_sch)
- sheet Power ports: added none; removed USB_DN, USB_DP
- note added: "Battery Connector"
- note added: "Connectors & Blocks"
- note added: "DEBUG"
- note added: "Output Terminal Block"
- note added: "Power Control"
- note added: "SWDIO"
- note added: "Speaker"
- note added: "USB"
- note added: "USB Input"
- note removed: "Audio Driver"
- note removed: "Flash"
- note removed: "IMU"
- note removed: "Terminal Block"
- moved on the sheet: C?, J1, J?, Q?, R?

Commit message: Added BOM parts, need to make new library part for LED
Parts:
- C101, C103: renamed from C?; footprint (none) -> Capacitor_SMD:C_0603_1608Metric; LCSC PN (none) -> C19702; MPN (none) -> CL10A106KP8NNNC
- C102: renamed from C?; footprint (none) -> Capacitor_SMD:C_0402_1005Metric; LCSC PN (none) -> C77020; MPN (none) -> GRM155R71H104KE14D
- C104, C105: renamed from C?; footprint (none) -> Capacitor_SMD:C_0603_1608Metric; LCSC PN (none) -> C2762594; MPN (none) -> CL10A226MO7JZNC
- J101: renamed from J?; footprint (none) -> TerminalBlock:TerminalBlock_Xinya_XY308-2.54-2P_1x02_P2.54mm_Horizontal; LCSC PN (none) -> C918120; MPN (none) -> DB125-2.54-2P-GN-S
- J102: renamed from J1; LCSC PN (none) -> C5118738; MPN (none) -> BM02B-ACHSS-GAN-ETF(LF)(SN)
- J103: renamed from J?; footprint (none) -> irex_Connector_USB:USB_C_Receptacle_GCT_USB4105-GF-A-060; LCSC PN (none) -> C963370; MPN (none) -> GT-USB-7010AN
- J104: renamed from J?; LCSC PN (none) -> C918123; MPN (none) -> DB125-2.54-5P-GN-S
- J105: renamed from J?; LCSC PN (none) -> C5155080
- J106: renamed from J?; LCSC PN (none) -> C5160786; MPN (none) -> DZ254S-11-03-48
- Q103: renamed from Q?; LCSC PN (none) -> C7431443; MPN (none) -> 2302V
- R101, R104, R105: renamed from R?; footprint (none) -> Resistor_SMD:R_0402_1005Metric; LCSC PN (none) -> C60490; MPN (none) -> RC0402FR-0710KL
- R102, R103: renamed from R?; footprint (none) -> Resistor_SMD:R_0402_1005Metric; LCSC PN (none) -> C105872; MPN (none) -> RC0402FR-075K1L
- R106: renamed from R?; footprint (none) -> Resistor_SMD:R_0402_1005Metric; LCSC PN (none) -> C106232; MPN (none) -> RC0402FR-07100RL
- TP101: renamed from TP?; now left out of the parts list
- U101: renamed from U?; footprint (none) -> Package_TO_SOT_SMD:SOT-143; LCSC PN (none) -> C19268160; MPN (none) -> CM1213A-02SR
- gave numbers to parts that had none: 3
Other:
- moved on the sheet: C101, J101, NT101

Commit message: Schematic finished, ready for layout
Parts:
- J104: footprint (none) -> TerminalBlock:TerminalBlock_Xinya_XY308-2.54-5P_1x05_P2.54mm_Horizontal
- J105: footprint (none) -> irex_Connector_Samtec:Samtec_FTSH-105-01-xxx-DV-K_2x05_P1.27mm_Vertical
- J106: footprint (none) -> Connector_PinHeader_2.54mm:PinHeader_1x03_P2.54mm_Vertical_SMD_Pin1Left
- NT101: footprint (none) -> NetTie:NetTie-2_SMD_Pad2.0mm
- Q101, Q102: footprint (none) -> Package_DFN_QFN:Diodes_UDFN2020-6_Type-F; symbol Device:Q_PMOS_GSD -> irex_Transistor_FET:XR25P01M
- Q103: footprint (none) -> Package_TO_SOT_SMD:SOT-23; symbol Device:Q_NMOS_GSD -> Transistor_FET:Q_NMOS_GSD
- TP101: footprint (none) -> TestPoint:TestPoint_THTPad_D2.0mm_Drill1.0mm
Connections:
- net VBAT_LED: now also Q101.4 (S), Q101.E2 (S), Q102.4 (S), Q102.E2 (S); no longer Q101.2 (S), Q102.2 (S)
- net VBAT_LED_SW: now also Q101.1 (D), Q101.2 (D), Q101.5 (D), Q101.6 (D), Q101.E1 (D), Q102.1 (D), Q102.2 (D), Q102.5 (D), Q102.6 (D), Q102.E1 (D); no longer Q101.3 (D), Q102.3 (D)
- net at Q103.3 (D), R104.1: now also Q101.3 (G), Q102.3 (G); no longer Q101.1 (G), Q102.1 (G)
Changed lines of the file:
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@@
 	)
 	(symbol
-		(lib_id "Device:Q_PMOS_GSD")
+		(lib_id "irex_Transistor_FET:XR25P01M")
 		(at 351.79 138.43 0)
 		(mirror x)
@@
 			)
 		)
-		(property "Footprint" ""
+		(property "Footprint" "Package_DFN_QFN:Diodes_UDFN2020-6_Type-F"
 			(at 356.87 140.97 0)
 			(effects
@@
 		)
 		(pin "3"
+		)
+		(pin "6"
+		)
+		(pin "E1"
+		)
+		(pin "4"
+		)
+		(pin "E2"
+		)
+		(pin "5"
 		)
 		(instances
@@
 			)
 		)
-		(property "Footprint" ""
+		(property "Footprint" "NetTie:NetTie-2_SMD_Pad2.0mm"
 			(at 92.71 39.37 0)
 			(effects
@@
 			)
 		)
-		(property "Footprint" ""
+		(property "Footprint" "irex_Connector_Samtec:Samtec_FTSH-105-01-xxx-DV-K_2x05_P1.27mm_Vertical"
 			(at 71.12 204.47 0)
 			(effects
@@
 	)
 	(symbol
-		(lib_id "Device:Q_NMOS_GSD")
+		(lib_id "Transistor_FET:Q_NMOS_GSD")
 		(at 331.47 148.59 0)
 		(unit 1)
@@
 			)
 		)
-		(property "Footprint" ""
+		(property "Footprint" "Package_TO_SOT_SMD:SOT-23"
 			(at 336.55 146.05 0)
 			(effects
@@
 			)
 		)
-		(property "Footprint" ""
+		(property "Footprint" "TestPoint:TestPoint_THTPad_D2.0mm_Drill1.0mm"
 			(at 191.77 58.42 0)
 			(effects
@@
 	)
 	(symbol
-		(lib_id "Device:Q_PMOS_GSD")
+		(lib_id "irex_Transistor_FET:XR25P01M")
 		(at 379.73 138.43 0)
 		(mirror x)
@@
 			)
 		)
-		(property "Footprint" ""
+		(property "Footprint" "Package_DFN_QFN:Diodes_UDFN2020-6_Type-F"
 			(at 384.81 140.97 0)
 			(effects
@@
 		)
 		(pin "3"
+		)
+		(pin "5"
+		)
+		(pin "6"
+		)
+		(pin "E1"
+		)
+		(pin "4"
+		)
+		(pin "E2"
 		)
 		(instances
@@
 			)
 		)
-		(property "Footprint" ""
+		(property "Footprint" "Connector_PinHeader_2.54mm:PinHeader_1x03_P2.54mm_Vertical_SMD_Pin1Left"
 			(at 72.39 224.79 0)
 			(effects
@@
 			)
 		)
-		(property "Footprint" ""
+		(property "Footprint" "TerminalBlock:TerminalBlock_Xinya_XY308-2.54-5P_1x05_P2.54mm_Horizontal"
 			(at 364.49 181.61 0)
 			(effects
