File: PCB Files/Power Core Board/Lightsaber Power Core/mcu_and_peripheral.kicad_sch (KiCad schematic)
At the start: 80 parts

Commit message: Added BOM parts, need to make new library part for LED
Parts:
- added TP301: PC14, symbol Connector:TestPoint
- C301, C302, C304, C310, C311, C315: renamed from C?; footprint (none) -> Capacitor_SMD:C_0402_1005Metric; LCSC PN (none) -> C77020; MPN (none) -> GRM155R71H104KE14D
- C303, C305, C306, C307, C308, C309, C313, C314: renamed from C?; footprint (none) -> Capacitor_SMD:C_0402_1005Metric; LCSC PN (none) -> C14445; MPN (none) -> CL05A105KP5NNNC
- C312: renamed from C?; footprint (none) -> Capacitor_SMD:C_0603_1608Metric; LCSC PN (none) -> C2762594; MPN (none) -> CL10A226MO7JZNC
- R301, R302, R308, R311, R314, R315: renamed from R?; footprint (none) -> Resistor_SMD:R_0402_1005Metric; LCSC PN (none) -> C60490; MPN (none) -> RC0402FR-0710KL
- R303, R307, R313: renamed from R?; footprint (none) -> Resistor_SMD:R_0402_1005Metric; LCSC PN (none) -> C60488; MPN (none) -> RC0402FR-072KL
- R304, R305, R306, R310: renamed from R?; footprint (none) -> Resistor_SMD:R_0402_1005Metric; LCSC PN (none) -> C106231; MPN (none) -> RC0402FR-070RL
- R309, R312, R316: renamed from R?; footprint (none) -> Resistor_SMD:R_0402_1005Metric; LCSC PN (none) -> C273705; MPN (none) -> RC0402FR-07634KL
- R317, R318, R319: renamed from R?; footprint (none) -> Resistor_SMD:R_0402_1005Metric; LCSC PN (none) -> C114764; MPN (none) -> RC0402FR-07200RL
- SW301, SW302: renamed from SW?; footprint (none) -> Button_Switch_SMD:SW_Push_SPST_NO_Alps_SKRK; LCSC PN (none) -> C720477; MPN (none) -> TS-1088-AR02016
- TP302, TP303, TP304, TP305, TP306, TP307, TP308: renamed from TP?; now left out of the parts list
- U301: renamed from U?; LCSC PN (none) -> C784817; MPN (none) -> LSM6DSRTR
- U302: renamed from U?; LCSC PN (none) -> C2943066; MPN (none) -> STM32L452CCU6
- U303: renamed from U?; footprint Package_BGA:WLP-9_1.448x1.468mm_Layout3x3_P0.4mm_Ball0.27mm_Pad0.25mm -> Package_DFN_QFN:TQFN-16-1EP_3x3mm_P0.5mm_EP1.23x1.23mm; LCSC PN (none) -> C910544; MPN (none) -> MAX98357AETE+T
- U304: renamed from U?; LCSC PN (none) -> C88868; MPN (none) -> W25N01GVZEIG
- gave numbers to parts that had none: 33
Connections:
- net PC14: now reaches U302.3 (PC14)
- net PC14: now also TP301.1

Commit message: Schematic finished, ready for layout
Parts:
- JP301, JP302: footprint (none) -> Jumper:SolderJumper-2_P1.3mm_Bridged2Bar_RoundedPad1.0x1.5mm
- TP301, TP302, TP303, TP304, TP305, TP306, TP307, TP308: footprint (none) -> TestPoint:TestPoint_Pad_D1.0mm
Changed lines of the file:
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@@
 			)
 		)
-		(property "Footprint" ""
+		(property "Footprint" "Jumper:SolderJumper-2_P1.3mm_Bridged2Bar_RoundedPad1.0x1.5mm"
 			(at 166.37 43.18 0)
 			(effects
@@
 			)
 		)
-		(property "Footprint" ""
+		(property "Footprint" "TestPoint:TestPoint_Pad_D1.0mm"
 			(at 81.28 132.08 0)
 			(effects
@@
 			)
 		)
-		(property "Footprint" ""
+		(property "Footprint" "TestPoint:TestPoint_Pad_D1.0mm"
 			(at 81.28 121.92 0)
 			(effects
@@
 			)
 		)
-		(property "Footprint" ""
+		(property "Footprint" "TestPoint:TestPoint_Pad_D1.0mm"
 			(at 81.28 134.62 0)
 			(effects
@@
 			)
 		)
-		(property "Footprint" ""
+		(property "Footprint" "Jumper:SolderJumper-2_P1.3mm_Bridged2Bar_RoundedPad1.0x1.5mm"
 			(at 128.27 43.18 0)
 			(effects
@@
 			)
 		)
-		(property "Footprint" ""
+		(property "Footprint" "TestPoint:TestPoint_Pad_D1.0mm"
 			(at 81.28 144.78 0)
 			(effects
@@
 			)
 		)
-		(property "Footprint" ""
+		(property "Footprint" "TestPoint:TestPoint_Pad_D1.0mm"
 			(at 170.18 109.22 0)
 			(effects
@@
 			)
 		)
+		(property "MPN" ""
+			(at 81.28 96.52 0)
+			(effects
+				(font
+					(size 1.27 1.27)
+				)
+				(hide yes)
+			)
+		)
 		(pin "1"
 		)
@@
 			)
 		)
-		(property "Footprint" ""
+		(property "Footprint" "TestPoint:TestPoint_Pad_D1.0mm"
 			(at 81.28 104.14 0)
 			(effects
@@
 			)
 		)
-		(property "Footprint" ""
+		(property "Footprint" "TestPoint:TestPoint_Pad_D1.0mm"
 			(at 81.28 116.84 0)
 			(effects
@@
 			)
 		)
-		(property "Footprint" ""
+		(property "Footprint" "TestPoint:TestPoint_Pad_D1.0mm"
 			(at 81.28 124.46 0)
 			(effects
